Commit message: Configure RGB-D camera and mapping launch for Map My World

File: urdf/my_robot.xacro (robot description, xacro)
@@ -141,4 +141,11 @@
   <axis xyz="0 1 0"/>
 </joint>
+  <joint name="camera_optical_joint" type="fixed">
+    <origin xyz="0 0 0" rpy="-1.5707 0 -1.5707"/>
+    <parent link="camera"/>
+    <child link="camera_link_optical"/>
+  </joint>
+  <link name="camera_link_optical">
+  </link>
 <!-- Hokuyo lidar link -->
 <link name="hokuyo">
